File: Hardware/Inverter.kicad_sch (KiCad schematic)
At the start: 56 parts, among them J2 Conn_01x02, J3 Conn_01x02, J4 Conn_01x01, J5 Conn_01x01, J6 Conn_01x01, Q1 WSD30100DN56, Q2 WSD30100DN56, Q3 WSD30100DN56, Q4 WSD30100DN56, Q5 WSD30100DN56, Q6 WSD30100DN56, U4 INA240A1PW, U5 LM321, U6 INA240A1PW, U7 INA240A1PW

Commit message: Update hardware exports and motor firmware
Parts:
- removed R13, R19, R23: 0.01R, Resistor_SMD:R_Shunt_Ohmite_LVK20, symbol Device:R_Shunt
- added R13, R19, R23: 0.01R, Resistor_SMD:R_2512_6332Metric, symbol Device:R
Connections:
- net OUT_A: now also U4.3 (-), R13.2
- net OUT_B: now also U6.3 (-), R19.2
- net OUT_C: now also U7.3 (-), R23.2
- net SHA: now also U4.2 (+), R13.1
- net SHB: now also U6.2 (+), R19.1
- net SHC: now also U7.2 (+), R23.1
