File: Hardware/foc_driver.kicad_pcb (KiCad board)
At the start: 2 copper layers, 60 x 56 mm, 132 parts, among them J1 Conn_01x03_MountingPin, J10 Conn_01x06_MountingPin, J11 Conn_01x05_MountingPin, J2 Conn_01x02, J3 Conn_01x02, J4 Conn_01x01, J5 Conn_01x01, J6 Conn_01x01, J7 USB_C_Receptacle_USB2.0_16P, J8 Conn_01x03_MountingPin, J9 Conn_01x03_MountingPin, Q1 WSD30100DN56, Q2 WSD30100DN56, Q3 WSD30100DN56, Q4 WSD30100DN56, Q5 WSD30100DN56, Q6 WSD30100DN56, U1 STM32F405RGTx, U10 AS5047D, U2 DRV8323RHRGZR, U3 LP2985-3.3, U4 INA240A1PW, U5 LM321, U6 INA240A1PW, U7 INA240A1PW, U8 USBLC6-2SC6, U9 TJA1051TK-3, Y1 12MHz

Commit message: Update hardware exports and motor firmware
Parts:
- R13, R19, R23: footprint Resistor_SMD:R_Shunt_Ohmite_LVK20 -> Resistor_SMD:R_2512_6332Metric
- moved R13 0.34 mm to (164.0, 104.5), turned to -90 degrees
- moved R19 0.34 mm to (164.0, 94.5), turned to -90 degrees
- moved R23 0.34 mm to (164.0, 84.5), turned to -90 degrees
Connections:
- R13 pad 2: Net-(U4-+) -> /Inverter/OUT_A
- R19 pad 2: Net-(U6-+) -> /Inverter/OUT_B
- R23 pad 2: Net-(U7-+) -> /Inverter/OUT_C
- U4 pad 2: Net-(U4-+) -> /Gate Driver/SHA
- U4 pad 3: Net-(U4--) -> /Inverter/OUT_A
- U6 pad 2: Net-(U6-+) -> /Gate Driver/SHB
- U6 pad 3: Net-(U6--) -> /Inverter/OUT_B
- U7 pad 2: Net-(U7-+) -> /Gate Driver/SHC
- U7 pad 3: Net-(U7--) -> /Inverter/OUT_C
Routing:
- net /Gate Driver/SHC: track 28.4 -> 40.1 mm, vias 6 -> 7
- net /Gate Driver/SHA: track 20.1 -> 31.4 mm, vias 6 -> 7
- net /Gate Driver/SHB: track 18.1 -> 29.5 mm, vias 6 -> 7
- net /Inverter/OUT_C: track 0.00 -> 10.1 mm, vias 0 -> 1
- net /Inverter/OUT_B: track 0.00 -> 10.1 mm, vias 0 -> 1
- net /Inverter/OUT_A: track 0.00 -> 10.1 mm, vias 0 -> 1
- net Net-(U6-+): track 9.77 -> 0.00 mm, vias 1 -> 0
- net Net-(U4-+): track 9.77 -> 0.00 mm, vias 1 -> 0
- net Net-(U7-+): track 9.68 -> 0.00 mm, vias 1 -> 0
- net Net-(U4--): track 8.18 -> 0.00 mm, vias 1 -> 0
- net Net-(U7--): track 8.09 -> 0.00 mm, vias 1 -> 0
- net Net-(U6--): track 8.09 -> 0.00 mm, vias 1 -> 0
- net /Gate Driver/GHC: track 25.5 -> 25.0 mm
Other:
- board text added: "Based on sf-motion Modified by MMU CYBERTRON Rev 1.0 - Yong Jun"
